Commit message: Door v4 in MuJoCo: upright, masses, passive hinge + handle spring, solid handle-frame collision, scene + manual control also made change to thumb base adn mujoko models

File: sw2+mujoko+python/output/Hand_forearm/urdf/Hand_forearm.urdf (robot description, URDF)
Before this commit: robot Hand_forearm, 18 links, 17 joints
Links:
- link human_hand_v3_2__Thumb_finger_1__Thumb_Base_1: mass 0.0146302 -> 0.0158405
Joints:
- joint human_hand_v3_2__Thumb_finger_1__Thumb_Base_1__human_hand_v3_2__Thumb_finger_1__Thumb_Proximal_1: axis -0.706872 0.024768 0.706907 -> 0 0.009285 0.999957; origin xyz=-0.0160461371 0.04490171905 0.01677608826 rpy=0 0 0 -> xyz=0.0008468628965 0.03322671905 0.03519308826 rpy=0 0 0
- joint human_hand_v3_2__Thumb_finger_1__Thumb_Proximal_1__human_hand_v3_2__Thumb_finger_1__Thumb_Distal_v2_1: axis -0.70687243 0.02476834 0.70690728 -> 0 0.00928507 0.99995689; origin xyz=0.0007980485926 0.03098864414 -0.0002873118661 rpy=0 0 0 -> xyz=0.0007983945436 0.03098793125 -0.0002878212196 rpy=0 0 0
- joint human_hand_v3_2__index_assem_2__Index_Middle_1__human_hand_v3_2__index_assem_2__Index_Distal_1: origin xyz=-0.02199270864 0.0005663384346 -5.258719644e-06 rpy=0 0 0 -> xyz=-0.0151507144 0.01595098479 -0.0001481124218 rpy=0 0 0
- joint human_hand_v3_2__index_assem_2__Index_Proximal_1__human_hand_v3_2__index_assem_2__Index_Middle_1: origin xyz=-0.02685808462 0.02827674577 -0.0002625629295 rpy=0 0 0 -> xyz=0.001004006868 0.03898539378 -0.0003619977801 rpy=0 0 0
